Commit message: first commit

File: mm_hyu.urdf (robot description, URDF)
Before this commit: robot mm_hyu, 12 links, 11 joints
Joints:
- joint Arm_Joint_1: axis 0 1 0 -> 0 0 1; origin xyz=0 -0.3107 0 rpy=0 0 0 -> xyz=0 0 0.1007 rpy=0 0 0
- joint Arm_Joint_2: origin xyz=0 -0.054 0 rpy=0 0 0 -> xyz=0  0 0.054 rpy=0 0 0
- joint Arm_Joint_3: origin xyz=0 0 -0.1458 rpy=0 0 0 -> xyz=0  0 0.1458 rpy=0 0 0
- joint Arm_Joint_4: origin xyz=0 0 -0.1542 rpy=0 0 0 -> xyz=0 0 0.1542  rpy=0 0 0
- joint Arm_Joint_5: origin xyz=0 0 -0.1458 rpy=0 0 0 -> xyz=0 0 0.1458  rpy=0 0 0
- joint Arm_Joint_6: origin xyz=0 0 -0.1542 rpy=0 0 0 -> xyz=0 0 0.1542  rpy=0 0 0
- joint Arm_Joint_base_joint: axis (none) -> 0 0 1; origin xyz=0 0 0.12 rpy=-1.57 0 1.57 -> xyz=0.085 0 0.0765 rpy=0 0 1.57

File: right_sim.urdf (robot description, URDF)
Before this commit: robot hyuspa, 8 links, 7 joints
Joints:
- joint Arm_Joint_1: axis 0 1 0 -> 0 0 1; origin xyz=0 -0.3107 0 rpy=0 0 0 -> xyz=0 0 0.1007 rpy=0 0 0
- joint Arm_Joint_2: origin xyz=0 -0.054 0 rpy=0 0 0 -> xyz=0  0 0.054 rpy=0 0 0
- joint Arm_Joint_3: origin xyz=0 0 -0.1458 rpy=0 0 0 -> xyz=0  0 0.1458 rpy=0 0 0
- joint Arm_Joint_4: origin xyz=0 0 -0.1542 rpy=0 0 0 -> xyz=0 0 0.1542  rpy=0 0 0
- joint Arm_Joint_5: origin xyz=0 0 -0.1458 rpy=0 0 0 -> xyz=0 0 0.1458  rpy=0 0 0
- joint Arm_Joint_6: origin xyz=0 0 -0.1542 rpy=0 0 0 -> xyz=0 0 0.1542  rpy=0 0 0
- joint Arm_Joint_base_joint: axis (none) -> 0 0 1; origin xyz=0 0 0 rpy=-1.57 0 0 -> xyz=0 0 0 rpy=0 0 0
